Commit message: xarm spherized

File: assets/xarm6/xarm6_rs_spherized.urdf (robot description, URDF)
Before this commit: robot xarm6, 27 links, 26 joints
Links:
- link left_finger: geometry collision sphere radius=0.019; collision sphere radius=0.019
- link link1: geometry collision sphere radius=0.055; collision sphere radius=0.06142438468845244
- link link2: geometry collision sphere radius=0.053144640769369575; collision sphere radius=0.0544142135623731
- link link3: geometry collision sphere radius=0.049; collision sphere radius=0.05
- link link4: geometry collision sphere radius=0.04307572505442989; collision sphere radius=0.048
- link link5: geometry collision sphere radius=0.046; collision sphere radius=0.05
- link link_base: geometry collision sphere radius=0.05623931699330031; collision sphere radius=0.06041831946211072
- link link_eef: geometry collision sphere radius=0.025414213562373177; collision sphere radius=0.02641421356237308
- link right_finger: geometry collision sphere radius=0.019; collision sphere radius=0.019
- link xarm_gripper_base_link: geometry collision sphere radius=0.044; collision sphere radius=0.044

Commit message: ruff format

File: assets/xarm6/xarm6_rs_spherized.urdf (robot description, URDF)
Before this commit: robot xarm6, 27 links, 26 joints
Links:
- link left_finger: geometry visual mesh filename=meshes/left_finger.stl
- link link1: geometry visual mesh filename=meshes/link1.stl
- link link2: geometry collision sphere radius=0.062070600459784936; collision sphere radius=0.062070600459784936
- link link3: geometry collision sphere radius=0.05; collision sphere radius=0.06240589416193893
- link link4: geometry visual mesh filename=meshes/link4.stl
- link link5: geometry visual mesh filename=meshes/link5.stl
- link link_base: geometry visual mesh filename=meshes/link_base.stl
- link link_eef: geometry visual mesh filename=meshes/d435_with_cam_stand.stl
- link right_finger: geometry visual mesh filename=meshes/right_finger.stl
- link xarm_gripper_base_link: geometry visual mesh filename=meshes/base_link.stl
